File: kicad-global/MS20-VCF.kicad_sch (KiCad schematic)
At the start: 68 parts, among them J1 FilterCV1, J2 FilterOut1, J3 Conn_CircuitBoard, J4 Conn_JackBoard, J5 FilterIn1, J6 Conn_CircuitBoard, J7 Conn_JackBoard, J8 Power Input, Q1 BC559, Q2 BC559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

Commit message: fix issues and add guide
Parts:
- C1: value 10µF -> 10uF; Comment  (none) -> Electrolytic cap
- C10, C5: value 10µ -> 10uF; Comment  (none) -> Electrolytic cap
- CUTCV1: Comment  (none) -> Use a small one (trimmer type)
- Q1, Q2: Comment  (none) -> Substitute BC558
- ResLv1: Comment  (none) -> variable resistor
Changed lines of the file:
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@@
     (pin "15")
     (pin "16")
-    (pin "10")
-    (pin "9")
+  )
+  (symbol (lib_id "Amplifier_Operational:LM13700") (at 96.52 52.07 0) (unit 3)
+    (in_bom yes) (on_board yes)
+    (property "Reference" "U1" (id 0) (at 96.52 42.7482 0))
+    (property "Value" "LM13700" (id 1) (at 96.52 45.0596 0))
+    (property "Footprint" "Package_SO:SOIC-16_3.9x9.9mm_P1.27mm" (id 2) (at 88.9 51.435 0)
+      (effects (font (size 1.27 1.27)) hide)
+    )
+    (property "Datasheet" "http://www.ti.com/lit/ds/symlink/lm13700.pdf" (id 3) (at 88.9 51.435 0)
+      (effects (font (size 1.27 1.27)) hide)
+    )
     (pin "1")
     (pin "2")
@@
     (pin "4")
     (pin "5")
-    (pin "7")
-    (pin "8")
-    (pin "11")
-    (pin "6")
-  )
-  (symbol (lib_id "Amplifier_Operational:LM13700") (at 96.52 52.07 0) (unit 3)
-    (in_bom yes) (on_board yes)
-    (property "Reference" "U1" (id 0) (at 96.52 42.7482 0))
-    (property "Value" "LM13700" (id 1) (at 96.52 45.0596 0))
-    (property "Footprint" "Package_SO:SOIC-16_3.9x9.9mm_P1.27mm" (id 2) (at 88.9 51.435 0)
-      (effects (font (size 1.27 1.27)) hide)
-    )
-    (property "Datasheet" "http://www.ti.com/lit/ds/symlink/lm13700.pdf" (id 3) (at 88.9 51.435 0)
-      (effects (font (size 1.27 1.27)) hide)
-    )
-    (pin "12")
-    (pin "13")
-    (pin "14")
-    (pin "15")
-    (pin "16")
-    (pin "10")
-    (pin "9")
-    (pin "1")
-    (pin "2")
-    (pin "3")
-    (pin "4")
-    (pin "5")
-    (pin "7")
-    (pin "8")
-    (pin "11")
-    (pin "6")
   )
   (symbol (lib_id "Amplifier_Operational:LM13700") (at 190.5 52.07 0) (unit 2)
@@
       (effects (font (size 1.27 1.27)) hide)
     )
-    (pin "12")
-    (pin "13")
-    (pin "14")
-    (pin "15")
-    (pin "16")
     (pin "10")
     (pin "9")
-    (pin "1")
-    (pin "2")
-    (pin "3")
-    (pin "4")
-    (pin "5")
-    (pin "7")
-    (pin "8")
-    (pin "11")
-    (pin "6")
   )
   (symbol (lib_id "Amplifier_Operational:LM13700") (at 125.73 52.07 0) (unit 4)
@@
       (effects (font (size 1.27 1.27)) hide)
     )
-    (pin "12")
-    (pin "13")
-    (pin "14")
-    (pin "15")
-    (pin "16")
-    (pin "10")
-    (pin "9")
-    (pin "1")
-    (pin "2")
-    (pin "3")
-    (pin "4")
-    (pin "5")
     (pin "7")
     (pin "8")
-    (pin "11")
-    (pin "6")
   )
   (symbol (lib_id "Amplifier_Operational:TL072") (at 193.04 78.74 180) (unit 1)
@@
     (pin "2")
     (pin "3")
+  )
+  (symbol (lib_id "Amplifier_Operational:TL072") (at 138.43 100.33 180) (unit 2)
+    (in_bom yes) (on_board yes)
+    (property "Reference" "U2" (id 0) (at 137.16 104.14 0))
+    (property "Value" "TL072" (id 1) (at 137.16 106.68 0))
+    (property "Footprint" "Package_DIP:DIP-8_W7.62mm_Socket" (id 2) (at 138.43 100.33 0)
+      (effects (font (size 1.27 1.27)) hide)
+    )
+    (property "Datasheet" "http://www.ti.com/lit/ds/symlink/tl071.pdf" (id 3) (at 138.43 100.33 0)
+      (effects (font (size 1.27 1.27)) hide)
+    )
     (pin "5")
     (pin "6")
     (pin "7")
-    (pin "4")
-    (pin "8")
-  )
-  (symbol (lib_id "Amplifier_Operational:TL072") (at 138.43 100.33 180) (unit 2)
-    (in_bom yes) (on_board yes)
-    (property "Reference" "U2" (id 0) (at 137.16 104.14 0))
-    (property "Value" "TL072" (id 1) (at 137.16 106.68 0))
-    (property "Footprint" "Package_DIP:DIP-8_W7.62mm_Socket" (id 2) (at 138.43 100.33 0)
-      (effects (font (size 1.27 1.27)) hide)
-    )
-    (property "Datasheet" "http://www.ti.com/lit/ds/symlink/tl071.pdf" (id 3) (at 138.43 100.33 0)
-      (effects (font (size 1.27 1.27)) hide)
-    )
-    (pin "1")
-    (pin "2")
-    (pin "3")
-    (pin "5")
-    (pin "6")
-    (pin "7")
-    (pin "4")
-    (pin "8")
   )
   (symbol (lib_id "Device:R") (at 76.2 54.61 90) (unit 1)
@@
     (in_bom yes) (on_board yes)
     (property "Reference" "C1" (id 0) (at 207.01 48.133 90))
-    (property "Value" "10µF" (id 1) (at 207.01 50.4444 90))
+    (property "Value" "10uF" (id 1) (at 207.01 50.4444 90))
     (property "Footprint" "Capacitor_THT:CP_Radial_D5.0mm_P2.00mm" (id 2) (at 203.2 55.5752 0)
       (effects (font (size 1.27 1.27)) hide)
     )
     (property "Datasheet" "~" (id 3) (at 207.01 54.61 0)
+      (effects (font (size 1.27 1.27)) hide)
+    )
+    (property "Comment " "Electrolytic cap" (id 4) (at 207.01 54.61 0)
       (effects (font (size 1.27 1.27)) hide)
     )
@@
       (effects (font (size 1.27 1.27)) hide)
     )
+    (property "Comment " "Use a small one (trimmer type)" (id 4) (at 166.37 123.19 0)
+      (effects (font (size 1.27 1.27)) hide)
+    )
     (pin "1")
     (pin "2")
@@
       (effects (font (size 1.27 1.27)) (justify left) hide)
     )
+    (property "Comment " "Substitute BC558" (id 4) (at 101.6 114.3 0)
+      (effects (font (size 1.27 1.27)) hide)
+    )
     (pin "1")
     (pin "2")
@@
     (property "Datasheet" "https://www.onsemi.com/pub/Collateral/BC556BTA-D.pdf" (id 3) (at 120.65 114.3 0)
       (effects (font (size 1.27 1.27)) (justify left) hide)
+    )
+    (property "Comment " "Substitute BC558" (id 4) (at 120.65 114.3 0)
+      (effects (font (size 1.27 1.27)) hide)
     )
     (pin "1")
@@
       (effects (font (size 1.27 1.27)) (justify left))
     )
-    (property "Value" "10µ" (id 1) (at 100.1014 172.593 0)
+    (property "Value" "10uF" (id 1) (at 100.1014 172.593 0)
       (effects (font (size 1.27 1.27)) (justify left))
     )
@@
       (effects (font (size 1.27 1.27)) hide)
     )
+    (property "Comment " "Electrolytic cap" (id 4) (at 97.79 171.45 0)
+      (effects (font (size 1.27 1.27)) hide)
+    )
     (pin "1")
     (pin "2")
@@
       (effects (font (size 1.27 1.27)) (justify left))
     )
-    (property "Value" "10µ" (id 1) (at 100.1014 185.293 0)
+    (property "Value" "10uF" (id 1) (at 100.1014 185.293 0)
       (effects (font (size 1.27 1.27)) (justify left))
     )
@@
     )
     (property "Datasheet" "~" (id 3) (at 97.79 184.15 0)
+      (effects (font (size 1.27 1.27)) hide)
+    )
+    (property "Comment " "Electrolytic cap" (id 4) (at 97.79 184.15 0)
       (effects (font (size 1.27 1.27)) hide)
     )
@@
       (effects (font (size 1.27 1.27)) hide)
     )
+    (property "Comment " "variable resistor" (id 4) (at 195.58 93.98 0)
+      (effects (font (size 1.27 1.27)) hide)
+    )
     (pin "1")
     (pin "2")
@@
       (effects (font (size 1.27 1.27)) hide)
     )
-    (pin "12")
-    (pin "13")
-    (pin "14")
-    (pin "15")
-    (pin "16")
-    (pin "10")
-    (pin "9")
-    (pin "1")
-    (pin "2")
-    (pin "3")
-    (pin "4")
-    (pin "5")
-    (pin "7")
-    (pin "8")
     (pin "11")
     (pin "6")
@@
       (effects (font (size 1.27 1.27)) hide)
     )
-    (pin "1")
-    (pin "2")
-    (pin "3")
-    (pin "5")
-    (pin "6")
-    (pin "7")
     (pin "4")
     (pin "8")
@@
     )
     (path "/00000000-0000-0000-0000-000060355101"
-      (reference "C1") (unit 1) (value "10µF") (footprint "Capacitor_THT:CP_Radial_D5.0mm_P2.00mm")
+      (reference "C1") (unit 1) (value "10uF") (footprint "Capacitor_THT:CP_Radial_D5.0mm_P2.00mm")
     )
     (path "/00000000-0000-0000-0000-00006034f1fc"
@@
     )
     (path "/00000000-0000-0000-0000-0000614ba8d1"
-      (reference "C5") (unit 1) (value "10µ") (footprint "Capacitor_THT:CP_Radial_D5.0mm_P2.00mm")
+      (reference "C5") (unit 1) (value "10uF") (footprint "Capacitor_THT:CP_Radial_D5.0mm_P2.00mm")
     )
     (path "/ffd08406-5515-49b6-babc-99d6d2951d61"
@@
     )
     (path "/00000000-0000-0000-0000-0000614ba8d7"
-      (reference "C10") (unit 1) (value "10µ") (footprint "Capacitor_THT:CP_Radial_D5.0mm_P2.00mm")
+      (reference "C10") (unit 1) (value "10uF") (footprint "Capacitor_THT:CP_Radial_D5.0mm_P2.00mm")
     )
     (path "/42600cf4-ebc1-4776-8647-e9e68e89f8e5"
@@
     )
     (path "/00000000-0000-0000-0000-0000615732ed/00000000-0000-0000-0000-0000615c9730"
-      (reference "C15") (unit 1) (value "10µF") (footprint "Capacitor_THT:CP_Radial_D5.0mm_P2.00mm")
+      (reference "C15") (unit 1) (value "10uF") (footprint "Capacitor_THT:CP_Radial_D5.0mm_P2.00mm")
     )
     (path "/00000000-0000-0000-0000-0000615732ed/00000000-0000-0000-0000-0000615c971b"

Commit message: update worflow run condition + trimmer footprint update
Parts:
- ResLv1: value 5k -> 10k; footprint Potentiometer_THT:Potentiometer_Bourns_3386X_Horizontal -> Potentiometer_THT:Potentiometer_Bourns_3386C_Horizontal
- ResVol1: footprint Potentiometer_THT:Potentiometer_Bourns_3386X_Horizontal -> Potentiometer_THT:Potentiometer_Bourns_3386C_Horizontal
Changed lines of the file:
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@@
     (pin "15")
     (pin "16")
+    (pin "10")
+    (pin "9")
+    (pin "1")
+    (pin "2")
+    (pin "3")
+    (pin "4")
+    (pin "5")
+    (pin "7")
+    (pin "8")
+    (pin "11")
+    (pin "6")
   )
   (symbol (lib_id "Amplifier_Operational:LM13700") (at 96.52 52.07 0) (unit 3)
@@
       (effects (font (size 1.27 1.27)) hide)
     )
+    (pin "12")
+    (pin "13")
+    (pin "14")
+    (pin "15")
+    (pin "16")
+    (pin "10")
+    (pin "9")
     (pin "1")
     (pin "2")
@@
     (pin "4")
     (pin "5")
+    (pin "7")
+    (pin "8")
+    (pin "11")
+    (pin "6")
   )
   (symbol (lib_id "Amplifier_Operational:LM13700") (at 190.5 52.07 0) (unit 2)
@@
       (effects (font (size 1.27 1.27)) hide)
     )
+    (pin "12")
+    (pin "13")
+    (pin "14")
+    (pin "15")
+    (pin "16")
     (pin "10")
     (pin "9")
+    (pin "1")
+    (pin "2")
+    (pin "3")
+    (pin "4")
+    (pin "5")
+    (pin "7")
+    (pin "8")
+    (pin "11")
+    (pin "6")
   )
   (symbol (lib_id "Amplifier_Operational:LM13700") (at 125.73 52.07 0) (unit 4)
@@
       (effects (font (size 1.27 1.27)) hide)
     )
+    (pin "12")
+    (pin "13")
+    (pin "14")
+    (pin "15")
+    (pin "16")
+    (pin "10")
+    (pin "9")
+    (pin "1")
+    (pin "2")
+    (pin "3")
+    (pin "4")
+    (pin "5")
     (pin "7")
     (pin "8")
+    (pin "11")
+    (pin "6")
   )
   (symbol (lib_id "Amplifier_Operational:TL072") (at 193.04 78.74 180) (unit 1)
@@
     (pin "2")
     (pin "3")
+    (pin "5")
+    (pin "6")
+    (pin "7")
+    (pin "4")
+    (pin "8")
   )
   (symbol (lib_id "Amplifier_Operational:TL072") (at 138.43 100.33 180) (unit 2)
@@
       (effects (font (size 1.27 1.27)) hide)
     )
+    (pin "1")
+    (pin "2")
+    (pin "3")
     (pin "5")
     (pin "6")
     (pin "7")
+    (pin "4")
+    (pin "8")
   )
   (symbol (lib_id "Device:R") (at 76.2 54.61 90) (unit 1)
@@
       (effects (font (size 1.27 1.27)) (justify right))
     )
-    (property "Value" "5k" (id 1) (at 194.31 93.98 90)
+    (property "Value" "10k" (id 1) (at 194.31 93.98 90)
       (effects (font (size 1.27 1.27)) (justify right))
     )
-    (property "Footprint" "Potentiometer_THT:Potentiometer_Bourns_3386X_Horizontal" (id 2) (at 195.58 93.98 0)
+    (property "Footprint" "Potentiometer_THT:Potentiometer_Bourns_3386C_Horizontal" (id 2) (at 195.58 93.98 0)
       (effects (font (size 1.27 1.27)) hide)
     )
@@
       (effects (font (size 1.27 1.27)) hide)
     )
+    (pin "12")
+    (pin "13")
+    (pin "14")
+    (pin "15")
+    (pin "16")
+    (pin "10")
+    (pin "9")
+    (pin "1")
+    (pin "2")
+    (pin "3")
+    (pin "4")
+    (pin "5")
+    (pin "7")
+    (pin "8")
     (pin "11")
     (pin "6")
@@
       (effects (font (size 1.27 1.27)) hide)
     )
+    (pin "1")
+    (pin "2")
+    (pin "3")
+    (pin "5")
+    (pin "6")
+    (pin "7")
     (pin "4")
     (pin "8")
@@
       (effects (font (size 1.27 1.27)) (justify right))
     )
-    (property "Footprint" "Potentiometer_THT:Potentiometer_Bourns_3386X_Horizontal" (id 2) (at 176.53 93.98 0)
+    (property "Footprint" "Potentiometer_THT:Potentiometer_Bourns_3386C_Horizontal" (id 2) (at 176.53 93.98 0)
       (effects (font (size 1.27 1.27)) hide)
     )
@@
     )
     (path "/00000000-0000-0000-0000-0000615804ec"
-      (reference "ResLv1") (unit 1) (value "5k") (footprint "Potentiometer_THT:Potentiometer_Bourns_3386X_Horizontal")
+      (reference "ResLv1") (unit 1) (value "10k") (footprint "Potentiometer_THT:Potentiometer_Bourns_3386C_Horizontal")
     )
     (path "/00000000-0000-0000-0000-0000615732ed/00000000-0000-0000-0000-0000615c9890"
-      (reference "ResLv2") (unit 1) (value "3.3k") (footprint "Potentiometer_THT:Potentiometer_Bourns_3386X_Horizontal")
+      (reference "ResLv2") (unit 1) (value "3.3k") (footprint "Potentiometer_THT:Potentiometer_Bourns_3386C_Horizontal")
     )
     (path "/00000000-0000-0000-0000-0000616e3eb9"
-      (reference "ResVol1") (unit 1) (value "10k") (footprint "Potentiometer_THT:Potentiometer_Bourns_3386X_Horizontal")
+      (reference "ResVol1") (unit 1) (value "10k") (footprint "Potentiometer_THT:Potentiometer_Bourns_3386C_Horizontal")
     )
     (path "/00000000-0000-0000-0000-0000615732ed/00000000-0000-0000-0000-0000615c98c2"
-      (reference "ResVol2") (unit 1) (value "10k") (footprint "Potentiometer_THT:Potentiometer_Bourns_3386X_Horizontal")
+      (reference "ResVol2") (unit 1) (value "10k") (footprint "Potentiometer_THT:Potentiometer_Bourns_3386C_Horizontal")
     )
     (path "/00000000-0000-0000-0000-000060338cd7"

Commit message: update front panel and infos on components
Parts:
- CUTCV1: Comment  Use a small one (trimmer type) -> Use a small shaft (trimmer type)
- ResLv1: Comment  variable resistor -> Bourns 3386C
- ResVol1: Comment  (none) -> Bourns 3386C
- SW2: Comment  (none) -> SPST On-On

Commit message: update documentation + update repo layout
Parts:
- C1, C10, C5: Comment  Electrolytic cap -> (none)
- CUTCV1: footprint Synth:Pot-bourns-alpha -> Kicad-perso:Pot-bourns-alpha; Comment  Use a small shaft (trimmer type) -> (none)
- CUTOFF1, Res1: footprint Synth:Pot-bourns-alpha -> Kicad-perso:Pot-bourns-alpha
- H1, H2, H3, H4: now left out of the parts list
- J1, J2, J5: footprint Synth:Thonkiconn -> Kicad-perso:Thonkiconn
- Q1, Q2: Comment  Substitute BC558 -> (none); Comments (none) -> Substitute BC558
- ResLv1, ResVol1: Comment  Bourns 3386C -> (none); Comments (none) -> Use multi turn Cermet style 3296 pots
- SW1: footprint Synth:SW_DPDT_Toggle -> Kicad-perso:SW_DPDT_Toggle; Comment  DPDT Switch, On-Off-On -> (none); Comments (none) -> DPDT Switch, On-Off-On
- SW2: footprint Synth:SW_Toggle_Blue_wSlots -> Kicad-perso:SW_Toggle_Blue_wSlots; Comment  SPST On-On -> (none)
Other:
- company: (none) -> Bleep Sound
- title: (none) -> MS20 VCF double
Changed lines of the file:
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@@
 (kicad_sch (version 20230121) (generator eeschema)
   (paper "A4")
+  (title_block
+    (title "MS20 VCF double")
+    (date "2023-09-23")
+    (rev "1.0")
+    (company "Bleep Sound")
+  )
   (junction (at 121.92 177.8) (diameter 0) (color 0 0 0 0)
   )
@@
       (effects (font (size 1.27 1.27)))
     )
-    (property "Footprint" "Synth:SW_DPDT_Toggle" (at 48.26 72.39 0)
+    (property "Footprint" "Kicad-perso:SW_DPDT_Toggle" (at 48.26 72.39 0)
       (effects (font (size 1.27 1.27)) hide)
     )
-    (property "Datasheet" "~" (at 48.26 72.39 0)
+    (property "Datasheet" "https://www.taydaelectronics.com/mini-toggle-switch-1m-series-dpdt-on-on.html" (at 48.26 72.39 0)
       (effects (font (size 1.27 1.27)) hide)
     )
-    (property "Comment " "DPDT Switch, On-Off-On " (at 48.26 77.47 0)
+    (property "Comments" "DPDT Switch, On-Off-On" (at 48.26 77.47 0)
       (effects (font (size 1.27 1.27)) hide)
     )
@@
       (effects (font (size 1.27 1.27)) hide)
     )
-    (property "Comment " "Electrolytic cap" (at 207.01 54.61 0)
-      (effects (font (size 1.27 1.27)) hide)
-    )
     (pin "1")
     (pin "2")
@@
       (effects (font (size 1.27 1.27)) (justify right))
     )
-    (property "Footprint" "Synth:Pot-bourns-alpha" (at 236.22 81.28 0)
+    (property "Footprint" "Kicad-perso:Pot-bourns-alpha" (at 236.22 81.28 0)
       (effects (font (size 1.27 1.27)) hide)
     )
@@
       (effects (font (size 1.27 1.27)) (justify right))
     )
-    (property "Footprint" "Synth:Pot-bourns-alpha" (at 182.88 146.05 0)
+    (property "Footprint" "Kicad-perso:Pot-bourns-alpha" (at 182.88 146.05 0)
       (effects (font (size 1.27 1.27)) hide)
     )
@@
       (effects (font (size 1.27 1.27)) (justify right))
     )
-    (property "Footprint" "Synth:Pot-bourns-alpha" (at 166.37 123.19 0)
+    (property "Footprint" "Kicad-perso:Pot-bourns-alpha" (at 166.37 123.19 0)
       (effects (font (size 1.27 1.27)) hide)
     )
@@
       (effects (font (size 1.27 1.27)) hide)
     )
-    (property "Comment " "Use a small shaft (trimmer type)" (at 166.37 123.19 0)
-      (effects (font (size 1.27 1.27)) hide)
-    )
     (pin "1")
     (pin "2")
@@
       (effects (font (size 1.27 1.27)) (justify left) hide)
     )
-    (property "Comment " "Substitute BC558" (at 101.6 114.3 0)
+    (property "Comments" "Substitute BC558" (at 101.6 114.3 0)
       (effects (font (size 1.27 1.27)) hide)
     )
@@
       (effects (font (size 1.27 1.27)) (justify left) hide)
     )
-    (property "Comment " "Substitute BC558" (at 120.65 114.3 0)
+    (property "Comments" "Substitute BC558" (at 120.65 114.3 0)
       (effects (font (size 1.27 1.27)) hide)
     )
@@
       (effects (font (size 1.27 1.27)) hide)
     )
-    (property "Comment " "Electrolytic cap" (at 97.79 171.45 0)
-      (effects (font (size 1.27 1.27)) hide)
-    )
     (pin "1")
     (pin "2")
@@
       (effects (font (size 1.27 1.27)) hide)
     )
-    (property "Comment " "Electrolytic cap" (at 97.79 184.15 0)
-      (effects (font (size 1.27 1.27)) hide)
-    )
     (pin "1")
     (pin "2")
@@
       (effects (font (size 1.27 1.27)))
     )
-    (property "Footprint" "Synth:SW_Toggle_Blue_wSlots" (at 49.53 101.6 0)
-      (effects (font (size 1.27 1.27)) hide)
-    )
-    (property "Datasheet" "~" (at 49.53 101.6 0)
+    (property "Footprint" "Kicad-perso:SW_Toggle_Blue_wSlots" (at 49.53 101.6 0)
       (effects (font (size 1.27 1.27)) hide)
     )
-    (property "Comment " "SPST On-On" (at 49.53 101.6 0)
+    (property "Datasheet" "https://www.taydaelectronics.com/mini-toggle-switch-spdt-on-on.html" (at 49.53 101.6 0)
       (effects (font (size 1.27 1.27)) hide)
     )
@@
       (effects (font (size 1.27 1.27)))
     )
-    (property "Footprint" "Synth:Thonkiconn" (at 226.06 113.03 0)
+    (property "Footprint" "Kicad-perso:Thonkiconn" (at 226.06 113.03 0)
       (effects (font (size 1.27 1.27)) hide)
     )
@@
       (effects (font (size 1.27 1.27)))
     )
-    (property "Footprint" "Synth:Thonkiconn" (at 251.46 113.03 0)
+    (property "Footprint" "Kicad-perso:Thonkiconn" (at 251.46 113.03 0)
       (effects (font (size 1.27 1.27)) hide)
     )
@@
       (effects (font (size 1.27 1.27)))
     )
-    (property "Footprint" "Synth:Thonkiconn" (at 226.06 130.81 0)
+    (property "Footprint" "Kicad-perso:Thonkiconn" (at 226.06 130.81 0)
       (effects (font (size 1.27 1.27)) hide)
     )
@@
       (effects (font (size 1.27 1.27)) hide)
     )
-    (property "Datasheet" "~" (at 195.58 93.98 0)
+    (property "Datasheet" "https://www.taydaelectronics.com/potentiometer-variable-resistors/cermet-potentiometers/3296w/10k-ohm-trimmer-potentiometer-cermet-25-turns-3296w.html" (at 195.58 93.98 0)
       (effects (font (size 1.27 1.27)) hide)
     )
-    (property "Comment " "Bourns 3386C" (at 195.58 93.98 0)
+    (property "Comments" "Use multi turn Cermet style 3296 pots " (at 195.58 93.98 0)
       (effects (font (size 1.27 1.27)) hide)
     )
@@
   )
   (symbol (lib_id "Mechanical:MountingHole_Pad") (at 22.86 17.78 0) (unit 1)
-    (in_bom yes) (on_board yes) (dnp no)
+    (in_bom no) (on_board yes) (dnp no)
     (property "Reference" "H1" (at 25.4 16.5354 0)
       (effects (font (size 1.27 1.27)) (justify left))
@@
   )
   (symbol (lib_id "Mechanical:MountingHole_Pad") (at 27.94 22.86 0) (unit 1)
-    (in_bom yes) (on_board yes) (dnp no)
+    (in_bom no) (on_board yes) (dnp no)
     (property "Reference" "H2" (at 30.48 21.6154 0)
       (effects (font (size 1.27 1.27)) (justify left))
@@
   )
   (symbol (lib_id "Mechanical:MountingHole_Pad") (at 33.02 27.94 0) (unit 1)
-    (in_bom yes) (on_board yes) (dnp no)
+    (in_bom no) (on_board yes) (dnp no)
     (property "Reference" "H3" (at 35.56 26.6954 0)
       (effects (font (size 1.27 1.27)) (justify left))
@@
   )
   (symbol (lib_id "Mechanical:MountingHole_Pad") (at 38.1 33.02 0) (unit 1)
-    (in_bom yes) (on_board yes) (dnp no)
+    (in_bom no) (on_board yes) (dnp no)
     (property "Reference" "H4" (at 40.64 31.7754 0)
       (effects (font (size 1.27 1.27)) (justify left))
@@
       (effects (font (size 1.27 1.27)) hide)
     )
-    (property "Datasheet" "~" (at 176.53 93.98 0)
+    (property "Datasheet" "https://www.taydaelectronics.com/potentiometer-variable-resistors/cermet-potentiometers/3296w/10k-ohm-trimmer-potentiometer-cermet-25-turns-3296w.html" (at 176.53 93.98 0)
       (effects (font (size 1.27 1.27)) hide)
     )
-    (property "Comment " "Bourns 3386C" (at 176.53 93.98 0)
+    (property "Comments" "Use multi turn Cermet style 3296 pots " (at 176.53 93.98 0)
       (effects (font (size 1.27 1.27)) hide)
     )

Commit message: update version number + hole size on front panel
Parts:
- CUTCV1: Comments (none) -> Use trimmer style pots for CUTCV1 and 2
- J1: value FilterCV1 -> Jack
- J2: value FilterOut1 -> Jack
- J5: value FilterIn1 -> Jack
Changed lines of the file:
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@@
   (title_block
     (title "MS20 VCF double")
-    (date "2023-09-23")
-    (rev "1.0")
+    (date "2023-10-06")
+    (rev "1.4")
     (company "Bleep Sound")
   )
@@
       (effects (font (size 1.27 1.27)) hide)
     )
+    (property "Comments" "Use trimmer style pots for CUTCV1 and 2" (at 166.37 123.19 0)
+      (effects (font (size 1.27 1.27)) hide)
+    )
     (pin "1")
     (pin "2")
@@
       (effects (font (size 1.27 1.27)))
     )
-    (property "Value" "FilterCV1" (at 226.8728 109.6264 0)
+    (property "Value" "Jack" (at 226.8728 109.6264 0)
       (effects (font (size 1.27 1.27)))
     )
@@
       (effects (font (size 1.27 1.27)))
     )
-    (property "Value" "FilterOut1" (at 252.2728 109.6264 0)
+    (property "Value" "Jack" (at 252.2728 109.6264 0)
       (effects (font (size 1.27 1.27)))
     )
@@
       (effects (font (size 1.27 1.27)))
     )
-    (property "Value" "FilterIn1" (at 226.8728 127.4064 0)
-      (effects (font (size 1.27 1.27)))
-    )
+    (property "Value" "Jack" (at 226.8728 127.4064 0)
+      (effects (font (size 1.27 1.27)))
+    )
