File: kicad-global/MS20-VCF.kicad_sch (KiCad schematic)
At the start: 68 parts, among them J1 Jack, J2 Jack, J3 Conn_CircuitBoard, J4 Conn_JackBoard, J5 Jack, J6 Conn_CircuitBoard, J7 Conn_JackBoard, J8 Power Input, Q1 BC559, Q2 BC559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

Commit message: V2.0
new front panel layout
new normalisation for CV and in/out for bandpass filter
Parts:
- removed D7: LED-12V, LED_THT:LED_D4.0mm, symbol Device:LED
- removed FB1, FB2: 10R, Inductor_THT:L_Axial_L7.0mm_D3.3mm_P10.16mm_Horizontal_Fastron_MICC, symbol Device:Ferrite_Bead_Small
- removed J1, J2, J5: Jack, Kicad-perso:Thonkiconn, symbol Connector:AudioJack2_Switch
- removed R22: 2.2k, Resistor_THT:R_Axial_DIN0207_L6.3mm_D2.5mm_P10.16mm_Horizontal, symbol Device:R
- removed SW2: Bandpass, Kicad-perso:SW_Toggle_Blue_wSlots, symbol Switch:SW_SPDT
- added D14, D7: 1N5819, Diode_THT:D_DO-41_SOD81_P10.16mm_Horizontal, symbol Diode:1N5819
- added J1, J2, J5: jack, Kicad-perso:Thonkiconn, symbol Kicad-perso:AudioJack_Switch
- C1, C10, C5: Links (none) -> https://www.taydaelectronics.com/capacitors/electrolytic-ca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
- C11, C12, C13, C14, C2, C3, C4, C6, C7, C8, C9: Links (none) -> https://www.taydaelectronics.com/capacitors/monolithic-cera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
- CUTCV1, CUTOFF1, Res1: value 100k -> B100k; Links (none) -> https://www.thonk.co.uk/shop/alpha-9mm-pots/
- D1, D2, D3, D4, D5, D6: Links (none) -> https://www.taydaelectronics.com/1n4148-switching-signal-di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
- J8: Links (none) -> https://www.thonk.co.uk/shop/eurorack-diy-essentials/
- Q1, Q2: Links (none) -> https://www.taydaelectronics.com/bc558-bc558b-transistor-pn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
- R1, R10, R11, R12, R13, R14, R15, R16, R17, R18, R19, R2, R20, R21, R3, R4, R5, R6, R7, R8, R9: Links (none) -> https://www.taydaelectronics.com/resistors/1-4w-metal-film-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
- ResLv1, ResVol1: footprint Potentiometer_THT:Potentiometer_Bourns_3386C_Horizontal -> Potentiometer_THT:Potentiometer_Bourns_3296W_Vertical; Links (none) -> https://www.thonk.co.uk/shop/25-turn-trimmer-potentiometer/
- SW1: Links (none) -> https://www.taydaelectronics.com/mini-toggle-switch-dpdt-on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
- U1: Links (none) -> https://eu.mouser.com/c/semiconductors/amplifier-ics/transc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
- U2: Links (none) -> https://eu.mouser.com/ProductDetail/Texas-Instruments/TL072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
Connections:
- net CVIn is gone; now on net GND: CUTCV1.1
- net +12V: now also D7.1 (K)
- net -12V: now also D14.2 (A)
- net Filter2In: now also J2.TN
- net FilterIn: now also J5.T
- net FilterOut: now also J2.T
- net GND: now also Res1.1, J1.S, J2.S, J5.S; no longer CUTCV1.3, Res1.3
- net at R12.1: now also Res1.3; no longer Res1.1
- net at CUTOFF1.1: now also R21.2; no longer R19.1
- net at CUTOFF1.3: now also R19.1; no longer R21.2
- net at J8.10 (Pin_10), J8.9 (Pin_9): now also D7.2 (A)
- net at J8.1 (Pin_1), J8.2 (Pin_2): now also D14.1 (K)
- new net CV1In: CUTCV1.3, J1.T
- new net CV2In: J1.TN
- no-connect marks 15 -> 10
Other:
- moved on the sheet: CUTCV1, CUTOFF1, Res1
